File: GhostPAW/KiCad/GhostPAW.kicad_sch (KiCad schematic)
At the start: 48 parts, among them IC6 74LVC1G04GM,115, IC9 TPS22995RZFR, J2 54102-0164, J3 505110-1092, J4 505110-1292, SW2 CUS-13TB

Commit message: Updated boards to pre production
Connections:
- net GND: now also SW2.SH
Changed lines of the file:
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@@
 	(wire
 		(pts
+			(xy 140.97 46.99) (xy 142.24 46.99)
+		)
+		(stroke
+			(width 0)
+			(type default)
+		)
+	)
+	(wire
+		(pts
 			(xy 154.94 83.82) (xy 151.13 83.82)
 		)
@@
 		(pin "4"
 		)
+		(pin "SH"
+		)
 		(instances
 			(project ""
@@
 					(unit 1)
 				)
+			)
+		)
+	)
+	(symbol
+		(lib_id "power:GND")
+		(at 140.97 46.99 0)
+		(unit 1)
+		(exclude_from_sim no)
+		(in_bom yes)
+		(on_board yes)
+		(dnp no)
+		(fields_autoplaced yes)
+		(property "Reference" "#PWR030"
+			(at 140.97 53.34 0)
+			(effects
+				(font
+					(size 1.27 1.27)
+				)
+				(hide yes)
+			)
+		)
+		(property "Value" "GND"
+			(at 140.97 52.07 0)
+			(effects
+				(font
+					(size 1.27 1.27)
+				)
+			)
+		)
+		(property "Footprint" ""
+			(at 140.97 46.99 0)
+			(effects
+				(font
+					(size 1.27 1.27)
+				)
+				(hide yes)
+			)
+		)
+		(property "Datasheet" ""
+			(at 140.97 46.99 0)
+			(effects
+				(font
+					(size 1.27 1.27)
+				)
+				(hide yes)
+			)
+		)
+		(property "Description" "Power symbol creates a global label with name \"GND\" , ground"
+			(at 140.97 46.99 0)
+			(effects
+				(font
+					(size 1.27 1.27)
+				)
+				(hide yes)
+			)
+		)
+		(pin "1"
+		)
+		(instances
+			(project "GhostPAW"
+				(path "/0c461ae4-ef22-4515-a234-7dcdbd16ae6e"
+					(reference "#PWR030")
+					(unit 1)
+				)
